Commit message: Imported upstream version '2.2.0' of 'upstream'

File: rc_visard_description/urdf/rc_visard_160.xacro (robot description, xacro)
@@ -2,5 +2,5 @@
 <robot name="rc_visard_160" xmlns:xacro="http://ros.org/wiki/xacro">
   <xacro:macro name="rc_160" params="prefix parent *origin">
-    <joint name="${prefix}camera" type="fixed">
+    <joint name="${prefix}camera_joint" type="fixed">
       <parent link="${parent}"/>
       <child link="${prefix}camera"/>
@@ -9,13 +9,17 @@
     <link name="${prefix}camera">
       <visual>
-          <geometry>
-              <mesh filename="package://rc_visard_description/meshes/visual/rc_visard_160.dae"/>
-          </geometry>
+        <geometry>
+          <mesh filename="package://rc_visard_description/meshes/visual/rc_visard_160.dae"/>
+        </geometry>
       </visual>
       <collision>
-          <geometry>
-              <mesh filename="package://rc_visard_description/meshes/collision/rc_visard_160.stl"/>
-          </geometry>
+        <geometry>
+          <mesh filename="package://rc_visard_description/meshes/collision/rc_visard_160.stl"/>
+        </geometry>
       </collision>
+      <inertial>
+        <mass value="0.675"/>
+        <inertia ixx="1.53" ixy="0.0" ixz="2.3" iyy="11.2" iyz="0.0" izz="10.6"/>
+      </inertial>
     </link>
   <link name="${prefix}mounting"/>
@@ -26,3 +30,3 @@
   </joint>
   </xacro:macro>
-  </robot>
+</robot>

File: rc_visard_description/urdf/rc_visard_65.xacro (robot description, xacro)
@@ -10,12 +10,16 @@
       <visual>
         <geometry>
-            <mesh filename="package://rc_visard_description/meshes/visual/rc_visard_65.dae"/>
+          <mesh filename="package://rc_visard_description/meshes/visual/rc_visard_65.dae"/>
         </geometry>
       </visual>
       <collision>
         <geometry>
-            <mesh filename="package://rc_visard_description/meshes/collision/rc_visard_65.stl"/>
+          <mesh filename="package://rc_visard_description/meshes/collision/rc_visard_65.stl"/>
         </geometry>
       </collision>
+      <inertial>
+        <mass value="0.675"/>
+        <inertia ixx="1.3" ixy="0.0" ixz="0.85" iyy="2.9" iyz="0.0" izz="2.3"/>
+      </inertial>
     </link>
   <link name="${prefix}mounting"/>
